Commit message: correcting addresses

File: urdf/robot_base.urdf.xacro (robot description, xacro)
@@ -2,8 +2,8 @@
 <robot name="robot_base" xmlns:xacro="http://www.ros.org/wiki/xacro">
     <!--______________________________ include ______________________________-->
-    <xacro:include filename="$(find robot_description)/urdf/robot_essentials.urdf.xacro"/>
-    <xacro:include filename="$(find robot_description)/urdf/robot_properties.urdf.xacro"/>
-    <xacro:include filename="$(find robot_description)/urdf/gazebo_essentials.urdf.xacro"/>
-    <xacro:include filename="$(find robot_description)/urdf/sensors/kinect.urdf.xacro"/>
+    <xacro:include filename="$(find robot_navigation)/urdf/robot_essentials.urdf.xacro"/>
+    <xacro:include filename="$(find robot_navigation)/urdf/robot_properties.urdf.xacro"/>
+    <xacro:include filename="$(find robot_navigation)/urdf/gazebo_essentials.urdf.xacro"/>
+    <xacro:include filename="$(find robot_navigation)/urdf/sensors/kinect.urdf.xacro"/>
     <!--_____________________________ robot base ____________________________-->
     <link name='base_link'>

File: urdf/sensors/kinect.urdf.xacro (robot description, xacro)
@@ -1,6 +1,6 @@
 <?xml version="1.0"?>
 <robot name="sensor_kinect" xmlns:xacro="http://ros.org/wiki/xacro">
-    <!--xacro:include filename="$(find robot_description)/urdf/turtlebot_gazebo.urdf.xacro"/-->
-    <xacro:include filename="$(find robot_description)/urdf/robot_properties.urdf.xacro"/>
+    <!--xacro:include filename="$(find robot_navigation)/urdf/turtlebot_gazebo.urdf.xacro"/-->
+    <xacro:include filename="$(find robot_navigation)/urdf/robot_properties.urdf.xacro"/>
     <!-- Parameterised in part by the values in turtlebot_properties.urdf.xacro -->
     <xacro:macro name="sensor_kinect" params="parent">
@@ -26,5 +26,5 @@
                 <origin xyz="0 0 0" rpy="0 0 ${M_PI/2}"/>
                 <geometry>
-                    <mesh filename="package://robot_description/meshes/sensors/kinect.dae"/>
+                    <mesh filename="package://robot_navigation/meshes/sensors/kinect.dae"/>
                 </geometry>
             </visual>

Commit message: simulating kinect on gazebo and rviz

File: urdf/robot_base.urdf.xacro (robot description, xacro)
@@ -5,5 +5,5 @@
     <xacro:include filename="$(find robot_navigation)/urdf/robot_properties.urdf.xacro"/>
     <xacro:include filename="$(find robot_navigation)/urdf/gazebo_essentials.urdf.xacro"/>
-    <xacro:include filename="$(find robot_navigation)/urdf/sensors/kinect.urdf.xacro"/>
+    <xacro:include filename="$(find robot_navigation)/urdf/sensors/kinect_base.urdf.xacro"/>
     <!--_____________________________ robot base ____________________________-->
     <link name='base_link'>

File: urdf/robot_properties.urdf.xacro (robot description, xacro)
@@ -22,7 +22,7 @@
     <xacro:property name="front_caster_origin"      value=" ${(robot_base_xsize/2)-0.10} 0.00000 -0.05000"/>
     <!--__________________________ kinect constants _________________________-->
-    <xacro:property name="cam_px"                   value="-0.0870"/>
-    <xacro:property name="kinect_cam_py"            value="-0.0125"/>
-	<xacro:property name="cam_pz"                   value="0.28700"/>
+    <xacro:property name="cam_px"                   value="0.25000"/>
+    <xacro:property name="cam_py"                   value="0.00000"/>
+	<xacro:property name="cam_pz"                   value="0.07600"/>
 	<xacro:property name="cam_or"                   value="0.00000"/>
 	<xacro:property name="cam_op"                   value="0.00000"/>

File: urdf/sensors/kinect_base.urdf.xacro (robot description, xacro)
@@ -1,10 +1,11 @@
 <?xml version="1.0"?>
 <robot name="sensor_kinect" xmlns:xacro="http://ros.org/wiki/xacro">
-    <!--xacro:include filename="$(find robot_navigation)/urdf/turtlebot_gazebo.urdf.xacro"/-->
+    <xacro:include filename="$(find robot_navigation)/urdf/sensors/kinect_gazebo.urdf.xacro"/>
     <xacro:include filename="$(find robot_navigation)/urdf/robot_properties.urdf.xacro"/>
-    <!-- Parameterised in part by the values in turtlebot_properties.urdf.xacro -->
+    <!--_______________ Parameters in this part is defined by _______________-->
+    <!--_____________ the values in robot_properties.urdf.xacro _____________-->
     <xacro:macro name="sensor_kinect" params="parent">
         <joint name="camera_rgb_joint" type="fixed">
-            <origin xyz="${cam_px} ${kinect_cam_py} ${cam_pz}" rpy="${cam_or} ${cam_op} ${cam_oy}"/>
+            <origin xyz="${cam_px} ${cam_py} ${cam_pz}" rpy="${cam_or} ${cam_op} ${cam_oy}"/>
             <parent link="${parent}"/>
             <child link="camera_rgb_frame" />
@@ -18,5 +19,5 @@
         <link name="camera_rgb_optical_frame"/>
         <joint name="camera_joint" type="fixed">
-            <origin xyz="-0.031 ${-kinect_cam_py} -0.016" rpy="0 0 0"/>
+            <origin xyz="-0.031 ${-cam_py} -0.016" rpy="0 0 0"/>
             <parent link="camera_rgb_frame"/>
             <child link="camera_link"/>
@@ -44,9 +45,6 @@
             </inertial>
         </link>
-        <!-- The fixed joints & links below are usually published by static_transformers launched by the OpenNi launch
-        files. However, for Gazebo simulation we need them, so we add them here.
-        (Hence, don't publish them additionally!) -->
         <joint name="camera_depth_joint" type="fixed">
-            <origin xyz="0 ${2 * -kinect_cam_py} 0" rpy="0 0 0" />
+            <origin xyz="0 ${2 * -cam_py} 0" rpy="0 0 0" />
             <parent link="camera_rgb_frame" />
             <child link="camera_depth_frame" />
@@ -59,6 +57,6 @@
         </joint>
         <link name="camera_depth_optical_frame"/>
-        <!-- Kinect sensor for simulation -->
-        <!--xacro:turtlebot_sim_3dsensor/-->
+        <!--__________________ Kinect sensor for simulation _________________-->
+        <xacro:simulate_depthSensor/>
     </xacro:macro>
 </robot>
